File: kicad/ViridianShield.kicad_pcb (KiCad board)
At the start: 2 copper layers, 68.6 x 53.3 mm, 27 parts, among them P1 Power, P2 Analog, P3 Digital, P4 Digital, P5 CONN_01X01, P6 CONN_01X01, P7 CONN_01X01, P8 CONN_01X01, Q1 2N7000, SW2 D2-7_INPUT_SWITCHES, U1 SFH620A-1

Commit message: kicad: Shield design evolution
Parts:
- removed A0_IN: A0_INPUT, Connector_PinHeader_2.54mm:PinHeader_1x03_P2.54mm_Vertical
- removed DIP_SWITCH: INTERNAL_SWITCHES, Package_DIP:DIP-8_W7.62mm_LongPads
- added RV2: A0_INPUT, Connector_PinHeader_2.54mm:PinHeader_1x03_P2.54mm_Vertical, F.Cu at (162.6, 114.3)
- added SW1: INTERNAL_SWITCHES, Package_DIP:DIP-8_W7.62mm_LongPads, F.Cu at (134.4, 89.0)
- added SW5: RESET_SWITCH, Button_Switch_THT:SW_PUSH_6mm, F.Cu at (113.3, 75.1)
- Q1: footprint Package_TO_SOT_THT:TO-92_Inline -> Package_TO_SOT_THT:TO-92_Wide
- R1: value 4.7k -> 1.6k
- moved REF** 26.7 mm to (118.4, 98.6), turned to 90 degrees
- moved U1 21.9 mm to (149.9, 108.8)
- moved R1 18.5 mm to (153.4, 97.9), turned to 0 degrees
- moved R2 17.4 mm to (137.2, 102.6)
- moved REF** 14.5 mm to (118.4, 110.0), turned to 90 degrees
- moved Q1 13.5 mm to (130.0, 89.5), turned to 90 degrees
- moved J3 7.79 mm to (130.4, 110.7), turned to 180 degrees
- moved R3 7.02 mm to (145.8, 94.6)
- moved R4 6.54 mm to (157.5, 119.8), turned to 180 degrees
- moved SW4 4.71 mm to (165.1, 104.1), turned to 0 degrees
- moved RV1 4.01 mm to (157.5, 109.2)
- moved SW3 3.31 mm to (162.6, 94.0)
- moved RV3 2.04 mm to (167.6, 114.3)
- moved SW2 1.15 mm to (149.9, 84.1)
- renumbered TELEINFO to J1, POWER to J2, DAC_MODULE to J3, VIRIDIAN to J4, MANUAL_IN to RV1, A1_IN to RV3, MAIN_PWR to SW3, MANUAL_SW to SW4
Connections:
- J1 pad 1: /EDF_IN -> Net-(J1-Pad1)
- P1 pad 3: (no net) -> /RESET
- P2 pad 5: /SDA -> (no net)
- P2 pad 6: /SCL -> (no net)
- P3 pad 1: (no net) -> /SCL
- P3 pad 2: (no net) -> /SDA
- P3 pad 5: (no net) -> /D13
- P3 pad 6: (no net) -> /D12
- P3 pad 7: (no net) -> /D11
- P3 pad 8: (no net) -> /D10
- P3 pad 9: /D9 -> (no net)
- P4 pad 8: /D0(RX) -> (no net)
- Q1 pad 3: /TELEINFO_OUT -> /D8
- R1 pad 2: /TELEINFO_IN -> Net-(J1-Pad1)
- R3 pad 2: /TELEINFO_OUT -> /D8
Routing:
- net /RESET: track 0.00 -> 63.5 mm
- net /D0(RX): track 54.4 -> 0.00 mm
- net /EDF_IN: track 46.5 -> 0.00 mm
- net /D9: track 25.5 -> 0.00 mm
- net /TELEINFO_OUT: track 23.9 -> 0.00 mm
- net Net-(J1-Pad2): track 46.3 -> 22.4 mm
- net +5V: track 113.1 -> 94.3 mm
- net Net-(Q1-Pad2): track 39.1 -> 25.2 mm
- net /TELEINFO_IN: track 12.7 -> 0.00 mm
- net /MANUAL_OUTPUT: track 19.1 -> 8.67 mm
- net /D11: track 0.00 -> 9.60 mm
- net /D12: track 0.00 -> 9.60 mm
- net /D13: track 0.00 -> 8.98 mm
- net /D10: track 0.00 -> 8.77 mm
- net Net-(J1-Pad1): track 0.00 -> 7.32 mm
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Other:
- board text added: "A0"
- board text added: "A1"
- board text added: "AUTO"
- board text added: "D10_IN"
- board text added: "D11_IN"
- board text added: "D12_IN"
- board text added: "D13_IN"
- board text added: "DAC_CONNECTOR"
- board text added: "MAIN_PWR"
- board text added: "MAN"
- board text added: "MANUAL"
- board text added: "RESET"
- board text added: "VIRIDIAN SHIELD - V02 - MAT-CAB"
- board text removed: "D8_IN"
- board text removed: "D9_IN"
- board text removed: "EDF_IN"
- board text removed: "RX_IN"
- board text removed: "VIRIDIAN SHIELD - V01 - MAT-CAB"

Commit message: kicad: V02 Shield update
Parts:
- added P9: Conn_02x03_Odd_Even, Connector_PinHeader_2.54mm:PinHeader_2x03_P2.54mm_Vertical, F.Cu at (174.6, 95.9)
- SW2: value D2-7_INPUT_SWITCHES -> D2-6_INPUT_SWITCHES; footprint ViridianShield:PinHeader_2x06_P2.54mm_Vertical_OtherPinAlloc -> ViridianShield:PinHeader_2x04_P2.54mm_Vertical_OtherPinAlloc
- moved SW3 16.8 mm to (177.2, 85.7), turned to 180 degrees
- moved J1 16.7 mm to (185.4, 96.5)
- moved SW1 15.6 mm to (149.9, 87.6)
- moved J2 13.4 mm to (185.4, 80.8)
- moved R1 13.1 mm to (164.5, 104.9)
- moved SW4 12.9 mm to (177.2, 108.6)
- moved SW2 12.2 mm to (161.9, 85.7)
- moved J4 11.9 mm to (185.4, 113.0)
- moved Q1 10.2 mm to (139.7, 86.4)
- moved R2 7.37 mm to (137.2, 95.2)
- moved U1 4.23 mm to (153.0, 106.0)
- moved R3 3.33 mm to (144.8, 91.4)
- moved SW5 0.92 mm to (114.2, 74.8)
- moved RV1 0.90 mm to (156.8, 108.6)
- moved RV2 0.90 mm to (161.9, 113.7)
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Connections:
- P2 pad 3: (no net) -> /A2
- P2 pad 4: (no net) -> /A3
- P3 pad 5: /D13 -> (no net)
- P3 pad 6: /D12 -> (no net)
- P3 pad 7: /D11 -> (no net)
- P3 pad 8: /D10 -> (no net)
- P3 pad 9: (no net) -> /D9
- P4 pad 4: /D4 -> (no net)
- Q1 pad 3: /D8 -> /D9
- R3 pad 2: /D8 -> /D9
- SW1 pad 5: /D10 -> /A3
- SW1 pad 6: /D11 -> /A2
- SW1 pad 7: /D12 -> /D7
- SW1 pad 8: /D13 -> /D8
- SW2 pad 5: GND -> /D2
- SW2 pad 6: GND -> /D3
- SW2 pad 7: /D2 -> /D5
- SW2 pad 8: /D3 -> /D6
Routing:
- net /A2: track 0.00 -> 50.7 mm, vias 0 -> 1
- net /A3: track 0.00 -> 49.6 mm, vias 0 -> 1
- net /D8: track 29.4 -> 5.60 mm
- net +5V: track 94.3 -> 114.3 mm
- net Net-(J1-Pad2): track 22.4 -> 35.9 mm
- net /D9: track 0.00 -> 13.0 mm
- net /MANUAL_OUTPUT: track 8.67 -> 21.4 mm
- net Net-(J3-Pad1): track 37.4 -> 49.6 mm
- net /D4: track 10.1 -> 0.00 mm
- net /D11: track 9.60 -> 0.00 mm
- net /D12: track 9.60 -> 0.00 mm
- net /D13: track 8.98 -> 0.00 mm
- net /D10: track 8.77 -> 0.00 mm
- net Net-(J1-Pad1): track 7.32 -> 14.3 mm
- net /RESET: track 63.5 -> 68.4 mm
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Other:
- board size 68.6 x 53.3 mm -> 78.7 x 53.3 mm
- board text added: "A2_IN"
- board text added: "A3_IN"
- board text added: "D8_IN"
- board text added: "TELEINFO"
- board text removed: "D10_IN"
- board text removed: "D11_IN"
- board text removed: "D12_IN"
- board text removed: "D13_IN"
- board text removed: "D4_IN"
